Commit message: chore: update PX4 version to v1.15.4 and adjust compatibility notes in README

File: models/common/quadrotor_base.xacro (robot description, xacro)
@@ -8,5 +8,6 @@
 <robot xmlns:xacro="http://www.ros.org/wiki/xacro">
   <!-- Macro for a basic quadrotor -->
-  <xacro:macro name="quadrotor_base" params="name
+  <xacro:macro name="quadrotor_base"
+    params="name
                                         mass='1.0'
                                         ixx='0.03' ixy='0' ixz='0'
@@ -53,7 +54,7 @@
           </geometry>
           <material>
-              <ambient>0 1 0 1</ambient>
-              <diffuse>0 1 0 1</diffuse>
-              <specular>0 1 0 1</specular>
+            <ambient>0 1 0 1</ambient>
+            <diffuse>0 1 0 1</diffuse>
+            <specular>0 1 0 1</specular>
           </material>
         </visual>
@@ -88,5 +89,5 @@
               accel_noise_density="${accel_noise_density}"
               accel_random_walk="${accel_random_walk}"
-              accel_bias_correlation_time="${accel_bias_correlation_time}"/>
+              accel_bias_correlation_time="${accel_bias_correlation_time}" />
           </imu>
         </sensor>
@@ -127,7 +128,7 @@
           </geometry>
           <material>
-              <ambient>0 1 0 1</ambient>
-              <diffuse>0 1 0 1</diffuse>
-              <specular>0 1 0 1</specular>
+            <ambient>0 1 0 1</ambient>
+            <diffuse>0 1 0 1</diffuse>
+            <specular>0 1 0 1</specular>
           </material>
         </visual>
@@ -176,7 +177,7 @@
           </geometry>
           <material>
-              <ambient>0 1 0 1</ambient>
-              <diffuse>0 1 0 1</diffuse>
-              <specular>0 1 0 1</specular>
+            <ambient>0 1 0 1</ambient>
+            <diffuse>0 1 0 1</diffuse>
+            <specular>0 1 0 1</specular>
           </material>
         </visual>
@@ -207,27 +208,28 @@
       <!-- Rotors -->
       <xacro:rotor_macro rotor_id="0"
-                         pos_x="0.3535533905932738"
-                         pos_y="0.35355339059327373"
-                         direction="cw"
-                         max_motor_thrust="${max_motor_thrust}"/>
+        pos_x="0.3535533905932738"
+        pos_y="0.35355339059327373"
+        direction="cw"
+        max_motor_thrust="${max_motor_thrust}" />
       <xacro:rotor_macro rotor_id="1"
-                         pos_x="-0.35355339059327373"
-                         pos_y="0.3535533905932738"
-                         direction="ccw"
-                         max_motor_thrust="${max_motor_thrust}"/>
+        pos_x="-0.35355339059327373"
+        pos_y="0.3535533905932738"
+        direction="ccw"
+        max_motor_thrust="${max_motor_thrust}" />
       <xacro:rotor_macro rotor_id="2"
-                         pos_x="-0.35355339059327384"
-                         pos_y="-0.35355339059327373"
-                         direction="cw"
-                         max_motor_thrust="${max_motor_thrust}"/>
+        pos_x="-0.35355339059327384"
+        pos_y="-0.35355339059327373"
+        direction="cw"
+        max_motor_thrust="${max_motor_thrust}" />
       <xacro:rotor_macro rotor_id="3"
-                         pos_x="0.3535533905932737"
-                         pos_y="-0.35355339059327384"
-                         direction="ccw"
-                         max_motor_thrust="${max_motor_thrust}"/>
+        pos_x="0.3535533905932737"
+        pos_y="-0.35355339059327384"
+        direction="ccw"
+        max_motor_thrust="${max_motor_thrust}" />
     </model>
   </xacro:macro>
   <!-- Macro for a single axis IMU noise -->
-  <xacro:macro name="imu_axis_noise" params="stddev dynamic_bias_stddev dynamic_bias_correlation_time">
+  <xacro:macro name="imu_axis_noise"
+    params="stddev dynamic_bias_stddev dynamic_bias_correlation_time">
     <noise type="gaussian">
       <mean>0</mean>
@@ -238,5 +240,6 @@
   </xacro:macro>
   <!-- Macro for IMU sensor noise parameters -->
-  <xacro:macro name="imu_noise_params" params="gyro_noise_density='0.00018665'
+  <xacro:macro name="imu_noise_params"
+    params="gyro_noise_density='0.00018665'
                                               gyro_random_walk='3.8785e-05'
                                               gyro_bias_correlation_time='1000'
@@ -247,16 +250,16 @@
       <x>
         <xacro:imu_axis_noise stddev="${gyro_noise_density}"
-                             dynamic_bias_stddev="${gyro_random_walk}"
-                             dynamic_bias_correlation_time="${gyro_bias_correlation_time}"/>
+          dynamic_bias_stddev="${gyro_random_walk}"
+          dynamic_bias_correlation_time="${gyro_bias_correlation_time}" />
       </x>
       <y>
         <xacro:imu_axis_noise stddev="${gyro_noise_density}"
-                             dynamic_bias_stddev="${gyro_random_walk}"
-                             dynamic_bias_correlation_time="${gyro_bias_correlation_time}"/>
+          dynamic_bias_stddev="${gyro_random_walk}"
+          dynamic_bias_correlation_time="${gyro_bias_correlation_time}" />
       </y>
       <z>
         <xacro:imu_axis_noise stddev="${gyro_noise_density}"
-                             dynamic_bias_stddev="${gyro_random_walk}"
-                             dynamic_bias_correlation_time="${gyro_bias_correlation_time}"/>
+          dynamic_bias_stddev="${gyro_random_walk}"
+          dynamic_bias_correlation_time="${gyro_bias_correlation_time}" />
       </z>
     </angular_velocity>
@@ -264,16 +267,16 @@
       <x>
         <xacro:imu_axis_noise stddev="${accel_noise_density}"
-                             dynamic_bias_stddev="${accel_random_walk}"
-                             dynamic_bias_correlation_time="${accel_bias_correlation_time}"/>
+          dynamic_bias_stddev="${accel_random_walk}"
+          dynamic_bias_correlation_time="${accel_bias_correlation_time}" />
       </x>
       <y>
         <xacro:imu_axis_noise stddev="${accel_noise_density}"
-                             dynamic_bias_stddev="${accel_random_walk}"
-                             dynamic_bias_correlation_time="${accel_bias_correlation_time}"/>
+          dynamic_bias_stddev="${accel_random_walk}"
+          dynamic_bias_correlation_time="${accel_bias_correlation_time}" />
       </y>
       <z>
         <xacro:imu_axis_noise stddev="${accel_noise_density}"
-                             dynamic_bias_stddev="${accel_random_walk}"
-                             dynamic_bias_correlation_time="${accel_bias_correlation_time}"/>
+          dynamic_bias_stddev="${accel_random_walk}"
+          dynamic_bias_correlation_time="${accel_bias_correlation_time}" />
       </z>
     </linear_acceleration>
@@ -302,14 +305,14 @@
         </geometry>
         <material>
-            <xacro:if value="${direction == 'cw'}">
-              <ambient>0 0 1 1</ambient>
-              <diffuse>0 0 1 1</diffuse>
-              <specular>0 0 1 1</specular>
-            </xacro:if>
-            <xacro:if value="${direction == 'ccw'}">
-              <ambient>1 0 0 1</ambient>
-              <diffuse>1 0 0 1</diffuse>
-              <specular>1 0 0 1</specular>
-            </xacro:if>
+          <xacro:if value="${direction == 'cw'}">
+            <ambient>0 0 1 1</ambient>
+            <diffuse>0 0 1 1</diffuse>
+            <specular>0 0 1 1</specular>
+          </xacro:if>
+          <xacro:if value="${direction == 'ccw'}">
+            <ambient>1 0 0 1</ambient>
+            <diffuse>1 0 0 1</diffuse>
+            <specular>1 0 0 1</specular>
+          </xacro:if>
         </material>
       </visual>
@@ -348,5 +351,5 @@
     </joint>
     <plugin filename="gz-sim-multicopter-motor-model-system"
-            name="gz::sim::systems::MulticopterMotorModel">
+      name="gz::sim::systems::MulticopterMotorModel">
       <jointName>rotor_${rotor_id}_joint</jointName>
       <linkName>rotor_${rotor_id}</linkName>
