Commit message: Add tilted hexarotor and octorotor GPS models
Rotor macro gains optional tilt/azimuth mount angles (flat default keeps
existing models unchanged). New hexa_tilted_gps and octo_tilted_gps models
cant every rotor radially outward by 15 degrees, with matching PX4 airframe
files (custom CA rotor geometry incl. axis vectors, autostart 6663/6664).

File: models/common/quadrotor_base.xacro (robot description, xacro)
@@ -282,10 +282,13 @@
     </linear_acceleration>
   </xacro:macro>
-  <!-- Macro for a rotor -->
-  <xacro:macro name="rotor_macro" params="rotor_id pos_x pos_y direction max_motor_thrust='30.0'">
+  <!-- Macro for a rotor. Optional mount tilt: the rotor frame is rotated by yaw `azimuth`
+       then pitch `tilt` (radians), so a radial-outward tilt at a given arm azimuth is
+       azimuth=arm angle, tilt=cant angle; the thrust stays along the rotor frame z axis. -->
+  <xacro:macro name="rotor_macro"
+    params="rotor_id pos_x pos_y direction max_motor_thrust='30.0' tilt='0' azimuth='0'">
     <link name="rotor_${rotor_id}">
       <gravity>true</gravity>
       <self_collide>false</self_collide>
-      <pose>${pos_x} ${pos_y} 0.01 0 0 0</pose>
+      <pose>${pos_x} ${pos_y} 0.01 0 ${tilt} ${azimuth}</pose>
       <inertial>
         <mass>1e-9</mass>
